File: hardware/Keypad/Keypad.kicad_sch (KiCad schematic)
At the start: 7 parts, among them J5 Keypad1, SW3 RIGHT, SW4 LEFT, SW5 SET

Commit message: redesign pcb files
Parts:
- added Brd1: SSD1306, SSD1306:128x64OLED, symbol SSD1306-128x64_OLED:SSD1306
- added H4, H5, H6, H7: MountingHole, MountingHole:MountingHole_2.2mm_M2, symbol Mechanical:MountingHole
- added J2: LCD, Connector_PinHeader_2.54mm:PinHeader_1x04_P2.54mm_Vertical, symbol Connector:Conn_01x04_Pin
Connections:
- net +3V3: now also Brd1.2 (VCC), J2.2 (Pin_2)
- net GND: now also Brd1.1 (GND), J2.1 (Pin_1)
- new net SCK: Brd1.3 (SCL), J2.3 (Pin_3)
- new net SDA: Brd1.4 (SDA), J2.4 (Pin_4)
